Commit message: Commiting to move it to ubuntu

File: harkbot/hark.urdf (robot description, URDF)
Before this commit: robot Hark, 9 links, 8 joints
Links:
- removed link Hand_v2_1
- removed link Link1_v2_1
- removed link finger_v2_1
- removed link finger_v2__1__1
- removed link link2_v2_1
- removed link link3_v2_1
- removed link link4_v2_1
- removed link link5_v2_1
- added link Hand, mass 2.2197201602974554; collision mesh filename=/meshes/collision/Hand_v2_1.stl scale=0.001 0.001 0.001; visual mesh filename=/meshes/visual/Hand_v2_1.stl scale=0.001 0.001 0.001
- added link Link1, mass 3.55259145758094; collision mesh filename=/meshes/collision/Link1_v2_1.stl scale=0.001 0.001 0.001; visual mesh filename=/meshes/visual/Link1_v2_1.stl scale=0.001 0.001 0.001
- added link finger1, mass 0.653538155273753; collision mesh filename=/meshes/collision/finger_v2_1.stl scale=0.001 0.001 0.001; visual mesh filename=/meshes/visual/finger_v2_1.stl scale=0.001 0.001 0.001
- added link finger2, mass 0.6535381552737535; collision mesh filename=/meshes/collision/finger_v2__1__1.stl scale=0.001 0.001 0.001; visual mesh filename=/meshes/visual/finger_v2__1__1.stl scale=0.001 0.001 0.001
- added link link2, mass 4.329966529786294; collision mesh filename=/meshes/collision/link2_v2_1.stl scale=0.001 0.001 0.001; visual mesh filename=/meshes/visual/link2_v2_1.stl scale=0.001 0.001 0.001
- added link link3, mass 3.239056584746587; collision mesh filename=/meshes/collision/link3_v2_1.stl scale=0.001 0.001 0.001; visual mesh filename=/meshes/visual/link3_v2_1.stl scale=0.001 0.001 0.001
- added link link4, mass 1.7025158483719638; collision mesh filename=/meshes/collision/link4_v2_1.stl scale=0.001 0.001 0.001; visual mesh filename=/meshes/visual/link4_v2_1.stl scale=0.001 0.001 0.001
- added link link5, mass 0.6135827464240919; collision mesh filename=/meshes/collision/link5_v2_1.stl scale=0.001 0.001 0.001; visual mesh filename=/meshes/visual/link5_v2_1.stl scale=0.001 0.001 0.001
Joints:
- joint Revolute 1: child Link1_v2_1 -> Link1
- joint Revolute 2: child link2_v2_1 -> link2; parent Link1_v2_1 -> Link1
- joint Revolute 3: child link3_v2_1 -> link3; parent link2_v2_1 -> link2
- joint Revolute 4: child link4_v2_1 -> link4; parent link3_v2_1 -> link3
- joint Revolute 5: child link5_v2_1 -> link5; parent link4_v2_1 -> link4
- joint Revolute 6: child Hand_v2_1 -> Hand; parent link5_v2_1 -> link5
- joint Slider 7: child finger_v2_1 -> finger1; parent Hand_v2_1 -> Hand
- joint Slider 8: child finger_v2__1__1 -> finger2; parent Hand_v2_1 -> Hand
