Commit message: sarthak debugging session

File: arkbot/ark_bot.urdf (robot description, URDF)
Before this commit: robot ArkBot, 9 links, 8 joints
Joints:
- removed joint Slider 8

Commit message: demos and drivers

File: arkbot/ark_bot.urdf (robot description, URDF)
Before this commit: robot ArkBot, 9 links, 7 joints
Joints:
- added joint Slider 8: type prismatic, parent Hand, child finger2, origin xyz=0.005124 -0.0562 0.127614 rpy=0 0 0, axis 0.0 -1.0 0.0, limit lower=-0.0425 upper=0.0 effort=100 velocity=100, mimic joint=Slider 7 multiplier=-1.0
